Commit message: models/juno, models/lyra: @model; the URDF's link meshes written by exports.py
The URDFs reference 3MF/<link>.3mf, which each project's exports.py writes from
its link models; nothing else in either project writes a file.

Co-Authored-By: Claude Fable 5.1 <noreply@anthropic.com>

File: models/juno/juno.urdf (robot description, URDF)
Before this commit: robot juno, 29 links, 28 joints
Links:
- link ankle_link_left: geometry collision box size=0.054 0.046 0.079; visual mesh filename=3MF/ankle_link_left.3mf scale=0.001 0.001 0.001
- link ankle_link_right: geometry collision box size=0.054 0.046 0.079; visual mesh filename=3MF/ankle_link_right.3mf scale=0.001 0.001 0.001
- link bicep_left: geometry collision box size=0.056 0.076 0.181; visual mesh filename=3MF/bicep_left.3mf scale=0.001 0.001 0.001
- link bicep_right: geometry collision box size=0.056 0.076 0.181; visual mesh filename=3MF/bicep_right.3mf scale=0.001 0.001 0.001
- link foot_left: geometry collision box size=0.18 0.07 0.043; visual mesh filename=3MF/foot_left.3mf scale=0.001 0.001 0.001
- link foot_right: geometry collision box size=0.18 0.07 0.043; visual mesh filename=3MF/foot_right.3mf scale=0.001 0.001 0.001
- link forearm_left: geometry collision box size=0.062 0.052 0.181; visual mesh filename=3MF/forearm_left.3mf scale=0.001 0.001 0.001
- link forearm_right: geometry collision box size=0.062 0.052 0.181; visual mesh filename=3MF/forearm_right.3mf scale=0.001 0.001 0.001
- link hand_left: geometry collision box size=0.096933 0.066685 0.191575; visual mesh filename=3MF/hand_left.3mf scale=0.001 0.001 0.001
- link hand_right: geometry collision box size=0.096933 0.066685 0.191575; visual mesh filename=3MF/hand_right.3mf scale=0.001 0.001 0.001
- link head: geometry collision box size=0.124743 0.1372 0.1375; visual mesh filename=3MF/head.3mf scale=0.001 0.001 0.001
- link hip_bracket_left: geometry collision box size=0.1 0.07 0.094; visual mesh filename=3MF/hip_bracket_left.3mf scale=0.001 0.001 0.001
- link hip_bracket_right: geometry collision box size=0.1 0.07 0.094; visual mesh filename=3MF/hip_bracket_right.3mf scale=0.001 0.001 0.001
- link hip_carrier_left: geometry collision box size=0.076 0.078 0.14; visual mesh filename=3MF/hip_carrier_left.3mf scale=0.001 0.001 0.001
- link hip_carrier_right: geometry collision box size=0.076 0.078 0.14; visual mesh filename=3MF/hip_carrier_right.3mf scale=0.001 0.001 0.001
- link neck_collar: geometry collision box size=0.044 0.049 0.066; visual mesh filename=3MF/neck_collar.3mf scale=0.001 0.001 0.001
- link pelvis: geometry collision box size=0.11139 0.265 0.122; visual mesh filename=3MF/pelvis.3mf scale=0.001 0.001 0.001
- link shin_left: geometry collision box size=0.106 0.07206 0.37; visual mesh filename=3MF/shin_left.3mf scale=0.001 0.001 0.001
- link shin_right: geometry collision box size=0.106 0.07206 0.37; visual mesh filename=3MF/shin_right.3mf scale=0.001 0.001 0.001
- link shoulder_pod_left: geometry collision box size=0.092 0.077 0.14; visual mesh filename=3MF/shoulder_pod_left.3mf scale=0.001 0.001 0.001
- link shoulder_pod_right: geometry collision box size=0.092 0.079 0.14; visual mesh filename=3MF/shoulder_pod_right.3mf scale=0.001 0.001 0.001
- link thigh_left: geometry collision box size=0.116645 0.0996 0.379; visual mesh filename=3MF/thigh_left.3mf scale=0.001 0.001 0.001
- link thigh_right: geometry collision box size=0.116645 0.0996 0.379; visual mesh filename=3MF/thigh_right.3mf scale=0.001 0.001 0.001
- link torso: geometry collision box size=0.139496 0.264 0.328; visual mesh filename=3MF/torso.3mf scale=0.001 0.001 0.001
- link wrist_carrier_left: geometry collision box size=0.048 0.044 0.052; visual mesh filename=3MF/wrist_carrier_left.3mf scale=0.001 0.001 0.001
- link wrist_carrier_right: geometry collision box size=0.048 0.044 0.052; visual mesh filename=3MF/wrist_carrier_right.3mf scale=0.001 0.001 0.001
- link yaw_housing_left: geometry collision box size=0.058 0.07 0.07; visual mesh filename=3MF/yaw_housing_left.3mf scale=0.001 0.001 0.001
- link yaw_housing_right: geometry collision box size=0.058 0.07 0.07; visual mesh filename=3MF/yaw_housing_right.3mf scale=0.001 0.001 0.001

File: models/lyra/lyra.urdf (robot description, URDF)
Before this commit: robot lyra, 18 links, 17 joints
Links:
- link index_distal: geometry collision box size=0.0106 0.0113 0.0286; visual mesh filename=3MF/index_distal.3mf scale=0.001 0.001 0.001
- link index_middle: geometry collision box size=0.0168 0.0136 0.0382; visual mesh filename=3MF/index_middle.3mf scale=0.001 0.001 0.001
- link index_proximal: geometry collision box size=0.0184 0.0149 0.0577; visual mesh filename=3MF/index_proximal.3mf scale=0.001 0.001 0.001
- link middle_distal: geometry collision box size=0.010918 0.011639 0.030268; visual mesh filename=3MF/middle_distal.3mf scale=0.001 0.001 0.001
- link middle_middle: geometry collision box size=0.017196 0.013969 0.041566; visual mesh filename=3MF/middle_middle.3mf scale=0.001 0.001 0.001
- link middle_proximal: geometry collision box size=0.018844 0.015308 0.062111; visual mesh filename=3MF/middle_proximal.3mf scale=0.001 0.001 0.001
- link palm: geometry collision box size=0.08 0.046 0.11124; visual mesh filename=3MF/palm.3mf scale=0.001 0.001 0.001
- link pinky_distal: geometry collision box size=0.009328 0.009944 0.025428; visual mesh filename=3MF/pinky_distal.3mf scale=0.001 0.001 0.001
- link pinky_middle: geometry collision box size=0.015216 0.012124 0.031736; visual mesh filename=3MF/pinky_middle.3mf scale=0.001 0.001 0.001
- link pinky_proximal: geometry collision box size=0.016624 0.013268 0.047056; visual mesh filename=3MF/pinky_proximal.3mf scale=0.001 0.001 0.001
- link ring_distal: geometry collision box size=0.010282 0.010961 0.028932; visual mesh filename=3MF/ring_distal.3mf scale=0.001 0.001 0.001
- link ring_middle: geometry collision box size=0.016404 0.013231 0.038834; visual mesh filename=3MF/ring_middle.3mf scale=0.001 0.001 0.001
- link ring_proximal: geometry collision box size=0.017956 0.014492 0.057289; visual mesh filename=3MF/ring_proximal.3mf scale=0.001 0.001 0.001
- link thumb_base: geometry collision box size=0.0288 0.0192 0.014; visual mesh filename=3MF/thumb_base.3mf scale=0.001 0.001 0.001
- link thumb_distal: geometry collision box size=0.0292 0.0108 0.011; visual mesh filename=3MF/thumb_distal.3mf scale=0.001 0.001 0.001
- link thumb_metacarpal: geometry collision box size=0.0592 0.0184 0.0151; visual mesh filename=3MF/thumb_metacarpal.3mf scale=0.001 0.001 0.001
- link thumb_proximal: geometry collision box size=0.0418 0.017 0.0138; visual mesh filename=3MF/thumb_proximal.3mf scale=0.001 0.001 0.001
